File: PCB/DynoDeck/DynoDeck.kicad_sch (KiCad schematic)
At the start: 76 parts, among them J1 USB_C_Receptacle_USB2.0_16P, J2 PGRM, J3 CardKBConn, J4 E-paper, J5 HC-IPEX0125-01 (u.FL), J6 BWSMA-KWE-Z001 (SMA), J7 CardKBRef, SW1 QON, SW2 POWER, SW3 RESET, SW4 IO1, U1 BQ25895RTW, U2 USBLC6-2SC6, U3 SX1262IMLTRT, U4 TUSB320, U5 MD7218E33PC1, U6 E73-2G4M08S1C, U7 PE42422MLAA-Z, U8 PE42422MLAA-Z, Y1 OW7EL89CENUXK7YLC-32M, Y3 3N00032G33YC

Commit message: nRF52840 remapping
Connections:
- net DC: no longer U6.16 (P0.08)
- net DIO1: now also U6.20 (P0.12); no longer U6.18 (P0.04/AIN2)
- net MISO: now also U6.16 (P0.08); no longer U6.33 (P0.13)
- net MOSI: now also U6.15 (P0.05/AIN3); no longer U6.32 (P0.20)
- net SCK: now also U6.14 (P0.06); no longer U6.30 (P0.17)
- net SCL: no longer U6.14 (P0.06)
- net SDA: no longer U6.15 (P0.05/AIN3)
- net SxBUSY: now also U6.18 (P0.04/AIN2); no longer U6.17 (P1.09)
- net SxNSS: now also U6.12 (P0.26); no longer U6.22 (P0.07)
- net ~{SxRESET}: now also U6.17 (P1.09); no longer U6.38 (P1.02)
- no-connect marks 22 -> 20
Changed lines of the file:
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@@
 	)
 	(no_connect
-		(at 302.26 120.65)
-	)
-	(no_connect
 		(at 302.26 77.47)
 	)
@@
 	)
 	(no_connect
-		(at 302.26 102.87)
-	)
-	(no_connect
 		(at 194.31 172.72)
 	)
@@
 	(wire
 		(pts
+			(xy 302.26 120.65) (xy 309.88 120.65)
+		)
+		(stroke
+			(width 0)
+			(type default)
+		)
+	)
+	(wire
+		(pts
 			(xy 110.49 160.02) (xy 121.92 160.02)
 		)
@@
 	(wire
 		(pts
+			(xy 302.26 87.63) (xy 312.42 87.63)
+		)
+		(stroke
+			(width 0)
+			(type default)
+		)
+	)
+	(wire
+		(pts
 			(xy 134.62 102.87) (xy 134.62 105.41)
 		)
@@
 		)
 	)
+	(wire
+		(pts
+			(xy 254 120.65) (xy 264.16 120.65)
+		)
+		(stroke
+			(width 0)
+			(type default)
+		)
+	)
 	(polyline
 		(pts
@@
 	(wire
 		(pts
-			(xy 302.26 110.49) (xy 309.88 110.49)
-		)
-		(stroke
-			(width 0)
-			(type default)
-		)
-	)
-	(wire
-		(pts
 			(xy 280.67 46.99) (xy 295.91 46.99)
 		)
@@
 		)
 	)
-	(wire
-		(pts
-			(xy 302.26 105.41) (xy 309.88 105.41)
-		)
-		(stroke
-			(width 0)
-			(type default)
-		)
-	)
 	(polyline
 		(pts
@@
 	(wire
 		(pts
-			(xy 308.61 130.81) (xy 302.26 130.81)
-		)
-		(stroke
-			(width 0)
-			(type default)
-		)
-	)
-	(wire
-		(pts
-			(xy 302.26 90.17) (xy 312.42 90.17)
+			(xy 302.26 95.25) (xy 312.42 95.25)
 		)
 		(stroke
@@
 	(wire
 		(pts
-			(xy 302.26 128.27) (xy 308.61 128.27)
-		)
-		(stroke
-			(width 0)
-			(type default)
-		)
-	)
-	(wire
-		(pts
 			(xy 259.08 157.48) (xy 259.08 158.75)
 		)
@@
 	(wire
 		(pts
-			(xy 302.26 92.71) (xy 312.42 92.71)
+			(xy 182.88 118.11) (xy 187.96 118.11)
 		)
 		(stroke
@@
 	(wire
 		(pts
-			(xy 182.88 118.11) (xy 187.96 118.11)
+			(xy 172.72 82.55) (xy 177.8 82.55)
 		)
 		(stroke
@@
 	(wire
 		(pts
-			(xy 172.72 82.55) (xy 177.8 82.55)
+			(xy 120.65 96.52) (xy 114.3 96.52)
 		)
 		(stroke
@@
 	(wire
 		(pts
-			(xy 120.65 96.52) (xy 114.3 96.52)
+			(xy 316.23 39.37) (xy 323.85 39.37)
 		)
 		(stroke
@@
 		)
 	)
-	(wire
+	(polyline
 		(pts
-			(xy 316.23 39.37) (xy 323.85 39.37)
+			(xy 342.9 139.7) (xy 342.9 170.18)
 		)
 		(stroke
@@
 		)
 	)
-	(polyline
+	(wire
 		(pts
-			(xy 342.9 139.7) (xy 342.9 170.18)
+			(xy 302.26 102.87) (xy 312.42 102.87)
 		)
 		(stroke
@@
 	(wire
 		(pts
-			(xy 302.26 95.25) (xy 312.42 95.25)
+			(xy 240.03 46.99) (xy 243.84 46.99)
 		)
 		(stroke
@@
 	(wire
 		(pts
-			(xy 240.03 46.99) (xy 243.84 46.99)
+			(xy 182.88 120.65) (xy 187.96 120.65)
 		)
 		(stroke
@@
 	(wire
 		(pts
-			(xy 182.88 120.65) (xy 187.96 120.65)
+			(xy 302.26 125.73) (xy 309.88 125.73)
 		)
 		(stroke
@@
 	(wire
 		(pts
-			(xy 41.91 102.87) (xy 41.91 83.82)
+			(xy 302.26 130.81) (xy 309.88 130.81)
 		)
 		(stroke
@@
 	(wire
 		(pts
-			(xy 34.29 83.82) (xy 38.1 83.82)
+			(xy 41.91 102.87) (xy 41.91 83.82)
 		)
 		(stroke
@@
 	(wire
 		(pts
-			(xy 49.53 38.1) (xy 54.61 38.1)
+			(xy 34.29 83.82) (xy 38.1 83.82)
 		)
 		(stroke
@@
 	(wire
 		(pts
-			(xy 48.26 40.64) (xy 49.53 40.64)
+			(xy 49.53 38.1) (xy 54.61 38.1)
 		)
 		(stroke
@@
 	(wire
 		(pts
-			(xy 142.24 41.91) (xy 148.59 41.91)
+			(xy 48.26 40.64) (xy 49.53 40.64)
 		)
 		(stroke
@@
 	(wire
 		(pts
-			(xy 63.5 48.26) (xy 69.85 48.26)
+			(xy 142.24 41.91) (xy 148.59 41.91)
 		)
 		(stroke
@@
 	(wire
 		(pts
-			(xy 254 113.03) (xy 264.16 113.03)
+			(xy 63.5 48.26) (xy 69.85 48.26)
 		)
 		(stroke
@@
 	(wire
 		(pts
-			(xy 302.26 87.63) (xy 312.42 87.63)
-		)
-		(stroke
-			(width 0)
-			(type default)
-		)
-	)
-	(wire
-		(pts
 			(xy 127 22.86) (xy 127 24.13)
 		)
@@
 		)
 	)
-	(wire
-		(pts
-			(xy 302.26 125.73) (xy 308.61 125.73)
-		)
-		(stroke
-			(width 0)
-			(type default)
-		)
-	)
 	(polyline
 		(pts
@@
 	(wire
 		(pts
-			(xy 254 120.65) (xy 264.16 120.65)
-		)
-		(stroke
-			(width 0)
-			(type default)
-		)
-	)
-	(wire
-		(pts
 			(xy 193.04 49.53) (xy 193.04 48.26)
 		)
@@
 	(wire
 		(pts
-			(xy 302.26 113.03) (xy 309.88 113.03)
-		)
-		(stroke
-			(width 0)
-			(type default)
-		)
-	)
-	(wire
-		(pts
 			(xy 134.62 95.25) (xy 135.89 95.25)
 		)
@@
 	(wire
 		(pts
-			(xy 226.06 156.21) (xy 234.95 156.21)
+			(xy 302.26 128.27) (xy 309.88 128.27)
 		)
 		(stroke
@@
 	(wire
 		(pts
-			(xy 302.26 85.09) (xy 312.42 85.09)
+			(xy 226.06 156.21) (xy 234.95 156.21)
 		)
 		(stroke
@@
 	(wire
 		(pts
+			(xy 302.26 85.09) (xy 312.42 85.09)
+		)
+		(stroke
+			(width 0)
+			(type default)
+		)
+	)
+	(wire
+		(pts
 			(xy 172.72 115.57) (xy 187.96 115.57)
 		)
@@
 	(wire
 		(pts
+			(xy 302.26 90.17) (xy 312.42 90.17)
+		)
+		(stroke
+			(width 0)
+			(type default)
+		)
+	)
+	(wire
+		(pts
 			(xy 151.13 92.71) (xy 153.67 92.71)
 		)
@@
 	)
 	(label "DIO1"
-		(at 312.42 85.09 180)
+		(at 312.42 102.87 180)
 		(effects
 			(font
@@
 	)
 	(label "MOSI"
-		(at 309.88 113.03 180)
+		(at 312.42 87.63 180)
 		(effects
 			(font
@@
 	)
 	(label "OTG"
-		(at 308.61 128.27 180)
+		(at 309.88 128.27 180)
 		(effects
 			(font
@@
 	)
 	(label "~{CE}"
-		(at 308.61 130.81 180)
+		(at 309.88 130.81 180)
 		(effects
 			(font
@@
 	)
 	(label "MISO"
-		(at 309.88 105.41 180)
+		(at 312.42 95.25 180)
 		(effects
 			(font
@@
 	)
 	(label "DC"
-		(at 312.42 95.25 180)
+		(at 317.5 97.79 180)
 		(effects
 			(font
@@
 	)
 	(label "~{INT}"
-		(at 308.61 125.73 180)
+		(at 309.88 125.73 180)
 		(effects
 			(font
@@
 	)
 	(label "SxNSS"
-		(at 312.42 92.71 180)
+		(at 309.88 120.65 180)
 		(effects
 			(font
@@
 	)
 	(label "SCL"
-		(at 312.42 90.17 180)
+		(at 273.05 101.6 180)
 		(effects
 			(font
@@
 	)
 	(label "~{SxRESET}"
-		(at 264.16 113.03 180)
+		(at 264.16 120.65 180)
 		(effects
 			(font
@@
 	)
 	(label "SCK"
-		(at 309.88 110.49 180)
+		(at 312.42 90.17 180)
 		(effects
 			(font
@@
 	)
 	(label "SxBUSY"
-		(at 264.16 120.65 180)
+		(at 312.42 85.09 180)
 		(effects
 			(font
@@
 	)
 	(label "SDA"
-		(at 312.42 87.63 180)
+		(at 276.86 110.49 180)
 		(effects
 			(font

Commit message: Bit of routing of Screen
Connections:
- net DC: now also U6.36 (P1.00)
- net ENSS: now also U6.32 (P0.20); no longer U6.34 (P0.22)
- net RES: now also U6.33 (P0.13); no longer U6.28 (P0.15)
- net SWDCLK: now also J2.3 (Pin_3); no longer J2.2 (Pin_2)
- net SWDIO: now also J2.2 (Pin_2); no longer J2.3 (Pin_3)
- net USER1: now also U6.22 (P0.07); no longer U6.36 (P1.00)
Changed lines of the file:
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@@
 	(wire
 		(pts
+			(xy 302.26 92.71) (xy 312.42 92.71)
+		)
+		(stroke
+			(width 0)
+			(type default)
+		)
+	)
+	(wire
+		(pts
 			(xy 64.77 149.86) (xy 64.77 151.13)
 		)
@@
 	(wire
 		(pts
+			(xy 157.48 158.75) (xy 167.64 158.75)
+		)
+		(stroke
+			(width 0)
+			(type default)
+		)
+	)
+	(wire
+		(pts
 			(xy 41.91 129.54) (xy 50.8 129.54)
 		)
@@
 	(wire
 		(pts
+			(xy 302.26 113.03) (xy 312.42 113.03)
+		)
+		(stroke
+			(width 0)
+			(type default)
+		)
+	)
+	(wire
+		(pts
 			(xy 34.29 129.54) (xy 41.91 129.54)
 		)
@@
 		)
 	)
+	(wire
+		(pts
+			(xy 302.26 105.41) (xy 312.42 105.41)
+		)
+		(stroke
+			(width 0)
+			(type default)
+		)
+	)
 	(polyline
 		(pts
@@
 	(wire
 		(pts
-			(xy 302.26 107.95) (xy 309.88 107.95)
-		)
-		(stroke
-			(width 0)
-			(type default)
-		)
-	)
-	(wire
-		(pts
 			(xy 33.02 83.82) (xy 34.29 83.82)
 		)
@@
 	(wire
 		(pts
-			(xy 254 110.49) (xy 264.16 110.49)
-		)
-		(stroke
-			(width 0)
-			(type default)
-		)
-	)
-	(wire
-		(pts
 			(xy 59.69 88.9) (xy 55.88 88.9)
 		)
@@
 	(wire
 		(pts
-			(xy 52.07 95.25) (xy 52.07 96.52)
+			(xy 157.48 156.21) (xy 167.64 156.21)
 		)
 		(stroke
@@
 	(wire
 		(pts
-			(xy 92.71 143.51) (xy 92.71 144.78)
+			(xy 52.07 95.25) (xy 52.07 96.52)
 		)
 		(stroke
@@
 	(wire
 		(pts
-			(xy 157.48 158.75) (xy 167.64 158.75)
+			(xy 92.71 143.51) (xy 92.71 144.78)
 		)
 		(stroke
@@
 	(wire
 		(pts
+			(xy 254 110.49) (xy 264.16 110.49)
+		)
+		(stroke
+			(width 0)
+			(type default)
+		)
+	)
+	(wire
+		(pts
 			(xy 280.67 41.91) (xy 289.56 41.91)
 		)
@@
 	(wire
 		(pts
-			(xy 157.48 156.21) (xy 167.64 156.21)
-		)
-		(stroke
-			(width 0)
-			(type default)
-		)
-	)
-	(wire
-		(pts
 			(xy 127 24.13) (xy 127 31.75)
 		)
@@
 	(wire
 		(pts
-			(xy 302.26 115.57) (xy 309.88 115.57)
-		)
-		(stroke
-			(width 0)
-			(type default)
-		)
-	)
-	(wire
-		(pts
 			(xy 95.25 44.45) (xy 110.49 44.45)
 		)
@@
 	)
 	(label "SWDIO"
-		(at 157.48 158.75 0)
+		(at 157.48 156.21 0)
 		(effects
 			(font
@@
 	)
 	(label "USER1"
-		(at 264.16 110.49 180)
+		(at 312.42 92.71 180)
 		(effects
 			(font
@@
 	)
 	(label "DC"
-		(at 317.5 97.79 180)
+		(at 264.16 110.49 180)
 		(effects
 			(font
@@
 	)
 	(label "RES"
-		(at 309.88 107.95 180)
+		(at 312.42 105.41 180)
 		(effects
 			(font
@@
 	)
 	(label "SWDCLK"
-		(at 157.48 156.21 0)
+		(at 157.48 158.75 0)
 		(effects
 			(font
@@
 	)
 	(label "ENSS"
-		(at 309.88 115.57 180)
+		(at 312.42 113.03 180)
 		(effects
 			(font
